File: hardware/drake_10b/drake_10b.kicad_sch (KiCad schematic)
At the start: 19 parts, among them J1 Conn_02x02_Odd_Even, J8 Conn_01x04, U1 nRF52832-QFxx, Y1 Crystal_GND24

Commit message: revised production files
Parts:
- C11, C5: now left out of the parts list
- J1: now not fitted; now left out of the parts list
- J8: FT Position Offset (none) -> 0,1.651
- U1: FT Rotation Offset (none) -> 180
Connections:
- net LED_GREEN renamed LED_YELLOW
- net LED_RED renamed LED_WHITE
Other:
- sheet hmi ports: added LED_WHITE, LED_YELLOW; removed LED_BLUE, LED_GREEN
- note added: "J8 only needed when device used as bar lights"
Changed lines of the file:
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@@
     (stroke (width 0) (type default))
+  )
+  (text "J8 only needed when device used as bar lights" (at 231.14 165.1 0)
+    (effects (font (size 1.27 1.27)) (justify left bottom))
   )
   (text "0.8pF is extended part\nLCSC part numer is for 1.0pF type"
@@
     (effects (font (size 1.27 1.27)) (justify left bottom))
   )
-  (label "LED_RED" (at 127 114.3 0) (fields_autoplaced)
+  (label "LED_WHITE" (at 127 114.3 0) (fields_autoplaced)
     (effects (font (size 1.27 1.27)) (justify left bottom))
   )
@@
     (effects (font (size 1.27 1.27)) (justify left bottom))
   )
-  (label "LED_GREEN" (at 127 111.76 0) (fields_autoplaced)
+  (label "LED_YELLOW" (at 127 111.76 0) (fields_autoplaced)
     (effects (font (size 1.27 1.27)) (justify left bottom))
   )
@@
     )
     (property "LCSC" "C77540" (at 93.98 86.36 0)
+      (effects (font (size 1.27 1.27)) hide)
+    )
+    (property "FT Rotation Offset" "180" (at 93.98 86.36 0)
       (effects (font (size 1.27 1.27)) hide)
     )
@@
   )
   (symbol (lib_id "drake_10b:Conn_02x02_Odd_Even") (at 55.88 137.16 0) (unit 1)
-    (in_bom yes) (on_board yes) (dnp no) (fields_autoplaced)
+    (in_bom no) (on_board yes) (dnp yes) (fields_autoplaced)
     (property "Reference" "J1" (at 57.15 130.81 0)
       (effects (font (size 1.27 1.27)))
@@
   )
   (symbol (lib_id "drake_10b:C") (at 53.34 31.75 0) (unit 1)
-    (in_bom yes) (on_board yes) (dnp yes) (fields_autoplaced)
+    (in_bom no) (on_board yes) (dnp yes) (fields_autoplaced)
     (property "Reference" "C5" (at 57.15 30.48 0)
       (effects (font (size 1.27 1.27)) (justify left))
@@
   )
   (symbol (lib_id "drake_10b:C") (at 48.26 63.5 0) (unit 1)
-    (in_bom yes) (on_board yes) (dnp yes) (fields_autoplaced)
+    (in_bom no) (on_board yes) (dnp yes) (fields_autoplaced)
     (property "Reference" "C11" (at 52.07 62.23 0)
       (effects (font (size 1.27 1.27)) (justify left))
@@
     )
     (property "LCSC" "C262260" (at 259.08 148.59 0)
+      (effects (font (size 1.27 1.27)) hide)
+    )
+    (property "FT Position Offset" "0,1.651" (at 259.08 148.59 0)
       (effects (font (size 1.27 1.27)) hide)
     )
@@
       (effects (font (size 1.27 1.27)) (justify left top))
     )
-    (pin "LED_GREEN" input (at 213.36 129.54 180)
+    (pin "LED_YELLOW" input (at 213.36 129.54 180)
       (effects (font (size 1.27 1.27)) (justify left))
     )
@@
       (effects (font (size 1.27 1.27)) (justify left))
     )
-    (pin "LED_BLUE" input (at 213.36 132.08 180)
-      (effects (font (size 1.27 1.27)) (justify left))
-    )
+    (pin "LED_WHITE" input (at 213.36 132.08 180)
+      (effects (font (size 1.27 1.27)) (justify left))
+    )
