File: hardware/drake_10b/hmi.kicad_sch (KiCad schematic)
At the start: 10 parts, among them SW1 SW_Push, SW2 SW_Push, SW3 SW_Push, SW4 SW_Push

Commit message: revised production files
Parts:
- D5: value green -> yellow; LCSC C2986059 -> C89811
- D6: value blue -> white; LCSC C2986058 -> C2290
- R15: value 1k5 -> 3k3; LCSC C25867 -> C25890
- R16: value 470 -> 3k3; LCSC C25117 -> C25890
- R17: value 220 -> 1k5; LCSC C25091 -> C25867
Connections:
- net LED_BLUE renamed LED_WHITE
- net LED_GREEN renamed LED_YELLOW
Other:
- note added: "SW3 and SW4 are just dummy buttons when populated top side only, can be ommited when both sides are assembled"
Changed lines of the file:
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@@
     (stroke (width 0) (type default))
   )
+  (text "SW3 and SW4 are just dummy buttons when populated top side only,\ncan be ommited when both sides are assembled"
+    (at 72.39 93.98 0)
+    (effects (font (size 1.27 1.27)) (justify left bottom))
+  )
   (hierarchical_label "BUT_LEFT" (shape output) (at 60.96 60.96 180) (fields_autoplaced)
     (effects (font (size 1.27 1.27)) (justify right))
@@
     (effects (font (size 1.27 1.27)) (justify right))
   )
-  (hierarchical_label "LED_BLUE" (shape input) (at 139.7 48.26 180) (fields_autoplaced)
-    (effects (font (size 1.27 1.27)) (justify right))
-  )
-  (hierarchical_label "LED_GREEN" (shape input) (at 139.7 50.8 180) (fields_autoplaced)
+  (hierarchical_label "LED_WHITE" (shape input) (at 139.7 48.26 180) (fields_autoplaced)
+    (effects (font (size 1.27 1.27)) (justify right))
+  )
+  (hierarchical_label "LED_YELLOW" (shape input) (at 139.7 50.8 180) (fields_autoplaced)
     (effects (font (size 1.27 1.27)) (justify right))
   )
@@
       (effects (font (size 1.27 1.27)) (justify right))
     )
-    (property "Value" "220" (at 160.02 60.96 0)
+    (property "Value" "1k5" (at 160.02 60.96 0)
       (effects (font (size 1.27 1.27)) (justify right))
     )
@@
       (effects (font (size 1.27 1.27)) hide)
     )
-    (property "LCSC" "C25091" (at 162.56 59.69 0)
+    (property "LCSC" "C25867" (at 162.56 59.69 0)
       (effects (font (size 1.27 1.27)) hide)
     )
@@
       (effects (font (size 1.27 1.27)) (justify left))
     )
-    (property "Value" "470" (at 149.86 60.96 0)
+    (property "Value" "3k3" (at 149.86 60.96 0)
       (effects (font (size 1.27 1.27)) (justify left))
     )
@@
       (effects (font (size 1.27 1.27)) hide)
     )
-    (property "LCSC" "C25117" (at 152.4 59.69 0)
+    (property "LCSC" "C25890" (at 152.4 59.69 0)
       (effects (font (size 1.27 1.27)) hide)
     )
@@
       (effects (font (size 1.27 1.27)) (justify right))
     )
-    (property "Value" "green" (at 148.59 72.7075 90)
+    (property "Value" "yellow" (at 148.59 72.7075 90)
       (effects (font (size 1.27 1.27)) (justify right))
     )
@@
       (effects (font (size 1.27 1.27)) hide)
     )
-    (property "LCSC" "C2986059" (at 152.4 69.85 90)
+    (property "LCSC" "C89811" (at 152.4 69.85 90)
       (effects (font (size 1.27 1.27)) hide)
     )
@@
       (effects (font (size 1.27 1.27)) (justify right))
     )
-    (property "Value" "1k5" (at 139.7 60.96 0)
+    (property "Value" "3k3" (at 139.7 60.96 0)
       (effects (font (size 1.27 1.27)) (justify right))
     )
@@
       (effects (font (size 1.27 1.27)) hide)
     )
-    (property "LCSC" "C25867" (at 142.24 59.69 0)
+    (property "LCSC" "C25890" (at 142.24 59.69 0)
       (effects (font (size 1.27 1.27)) hide)
     )
@@
   (symbol (lib_id "drake_10b:LED") (at 162.56 69.85 270) (mirror x) (unit 1)
     (in_bom yes) (on_board yes) (dnp no) (fields_autoplaced)
-    (property "Reference" "D6" (at 158.75 70.1675 90)
-      (effects (font (size 1.27 1.27)) (justify right))
-    )
-    (property "Value" "blue" (at 158.75 72.7075 90)
-      (effects (font (size 1.27 1.27)) (justify right))
+    (property "Reference" "D6" (at 165.1 70.1675 90)
+      (effects (font (size 1.27 1.27)) (justify left))
+    )
+    (property "Value" "white" (at 165.1 72.7075 90)
+      (effects (font (size 1.27 1.27)) (justify left))
     )
     (property "Footprint" "Library:LED_0603_1608Metric" (at 162.56 69.85 0)
@@
       (effects (font (size 1.27 1.27)) hide)
     )
-    (property "LCSC" "C2986058" (at 162.56 69.85 90)
-      (effects (font (size 1.27 1.27)) hide)
-    )
+    (property "LCSC" "C2290" (at 162.56 69.85 90)
+      (effects (font (size 1.27 1.27)) hide)
+    )
