File: hardware/drake_10b/i2c.kicad_sch (KiCad schematic)
At the start: 9 parts, among them J5 Conn_01x04, J6 Conn_01x04, U4 LIS2DH12TR

Commit message: revised production files
Parts:
- D21, D54: FT Rotation Offset (none) -> 180
- J5: FT Position Offset (none) -> 0,1.651
- J6: LT Position Offset (none) -> 0,1.651
Other:
- note added: "J5 only populated when using device as actuator or 16 LED taillight"
- note added: "J6 only populated when using device as actuator"
Changed lines of the file:
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@@
     (stroke (width 0) (type default))
+  )
+  (text "J6 only populated when using\ndevice as actuator" (at 149.86 44.45 0)
+    (effects (font (size 1.27 1.27)) (justify left bottom))
+  )
+  (text "J5 only populated when using device\nas actuator or 16 LED taillight"
+    (at 73.66 43.18 0)
+    (effects (font (size 1.27 1.27)) (justify left bottom))
   )
   (hierarchical_label "SCL_IN" (shape input) (at 121.92 48.26 180) (fields_autoplaced)
@@
     )
     (property "LCSC" "C262260" (at 64.77 45.72 0)
+      (effects (font (size 1.27 1.27)) hide)
+    )
+    (property "FT Position Offset" "0,1.651" (at 64.77 45.72 0)
       (effects (font (size 1.27 1.27)) hide)
     )
@@
       (effects (font (size 1.27 1.27)) hide)
     )
+    (property "LT Position Offset" "0,1.651" (at 140.97 45.72 0)
+      (effects (font (size 1.27 1.27)) hide)
+    )
     (pin "2")
     (pin "3")
@@
       (effects (font (size 1.27 1.27)) hide)
     )
+    (property "FT Rotation Offset" "180" (at 127 55.88 90)
+      (effects (font (size 1.27 1.27)) hide)
+    )
     (pin "1")
     (pin "3")
@@
       (effects (font (size 1.27 1.27)) hide)
     )
+    (property "FT Rotation Offset" "180" (at 50.8 55.88 90)
+      (effects (font (size 1.27 1.27)) hide)
+    )
