File: hardware/drake_10b/motor.kicad_sch (KiCad schematic)
At the start: 15 parts, among them J10 Conn_01x04, J4 Conn_01x01, J7 Conn_01x01, J9 Conn_01x04, U5 BDR6125, U6 ITR8307-S18-TR8

Commit message: revised production files
Parts:
- C68: footprint Capacitor_SMD:C_0402_1005Metric -> Library:C_0402_1005Metric
- J10: footprint rt_connectors:FFC_SolderCon_4pin_3,5x0,3mm_Pitch0.5mm -> Library:FFC_SolderCon_4pin_3,5x0,3mm_Pitch0.5mm; now left out of the parts list
- J4, J7, J9: now left out of the parts list
- R13: value 82k -> 75k; footprint Resistor_SMD:R_0402_1005Metric -> Library:R_0402_1005Metric; JLC 0603 -> 0402; LCSC C22843 -> C25798
- R14, R18: footprint Resistor_SMD:R_0402_1005Metric -> Library:R_0402_1005Metric; JLC 0603 -> 0402; LCSC C22843 -> C25867
- U5: footprint Package_SO:SOIC-8_3.9x4.9mm_P1.27mm -> Library:SOIC-8_3.9x4.9mm_P1.27mm
- U6: FT Rotation Offset (none) -> -90
Changed lines of the file:
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@@
   )
   (symbol (lib_id "drake_10b:Conn_01x01") (at 93.98 71.12 0) (unit 1)
-    (in_bom yes) (on_board yes) (dnp no) (fields_autoplaced)
+    (in_bom no) (on_board yes) (dnp no) (fields_autoplaced)
     (property "Reference" "J7" (at 96.52 69.85 0)
       (effects (font (size 1.27 1.27)) (justify left))
@@
   )
   (symbol (lib_id "drake_10b:Conn_01x04") (at 182.88 29.21 0) (unit 1)
-    (in_bom yes) (on_board yes) (dnp no)
+    (in_bom no) (on_board yes) (dnp no)
     (property "Reference" "J10" (at 185.42 29.21 0)
       (effects (font (size 1.27 1.27)) (justify left))
@@
       (effects (font (size 1.27 1.27)) (justify left))
     )
-    (property "Footprint" "rt_connectors:FFC_SolderCon_4pin_3,5x0,3mm_Pitch0.5mm" (at 182.88 29.21 0)
+    (property "Footprint" "Library:FFC_SolderCon_4pin_3,5x0,3mm_Pitch0.5mm" (at 182.88 29.21 0)
       (effects (font (size 1.27 1.27)) hide)
     )
@@
       (effects (font (size 1.27 1.27)) hide)
     )
+    (property "FT Rotation Offset" "-90" (at 149.86 78.74 0)
+      (effects (font (size 1.27 1.27)) hide)
+    )
     (pin "3")
     (pin "2")
@@
       (effects (font (size 1.27 1.27)) (justify right))
     )
-    (property "Value" "82k" (at 134.62 73.66 0)
+    (property "Value" "75k" (at 134.62 73.66 0)
       (effects (font (size 1.27 1.27)) (justify right))
     )
-    (property "Footprint" "Resistor_SMD:R_0402_1005Metric" (at 133.35 74.422 90)
+    (property "Footprint" "Library:R_0402_1005Metric" (at 133.35 74.422 90)
       (effects (font (size 1.27 1.27)) hide)
     )
@@
       (effects (font (size 1.27 1.27)) hide)
     )
-    (property "JLC" "0603" (at 133.35 76.2 0)
-      (effects (font (size 1.27 1.27)) hide)
-    )
-    (property "LCSC" "C22843" (at 133.35 76.2 0)
+    (property "JLC" "0402" (at 133.35 76.2 0)
+      (effects (font (size 1.27 1.27)) hide)
+    )
+    (property "LCSC" "C25798" (at 133.35 76.2 0)
       (effects (font (size 1.27 1.27)) hide)
     )
@@
       (effects (font (size 1.27 1.27)) (justify left))
     )
-    (property "Footprint" "Package_SO:SOIC-8_3.9x4.9mm_P1.27mm" (at 50.8 78.74 0)
+    (property "Footprint" "Library:SOIC-8_3.9x4.9mm_P1.27mm" (at 50.8 78.74 0)
       (effects (font (size 1.27 1.27)) hide)
     )
@@
   )
   (symbol (lib_id "drake_10b:Conn_01x04") (at 182.88 41.91 0) (unit 1)
-    (in_bom yes) (on_board yes) (dnp no)
+    (in_bom no) (on_board yes) (dnp no)
     (property "Reference" "J9" (at 185.42 41.91 0)
       (effects (font (size 1.27 1.27)) (justify left))
@@
   )
   (symbol (lib_id "drake_10b:Conn_01x01") (at 93.98 55.88 0) (unit 1)
-    (in_bom yes) (on_board yes) (dnp no) (fields_autoplaced)
+    (in_bom no) (on_board yes) (dnp no) (fields_autoplaced)
     (property "Reference" "J4" (at 96.52 54.61 0)
       (effects (font (size 1.27 1.27)) (justify left))
@@
       (effects (font (size 1.27 1.27)) (justify left))
     )
-    (property "Footprint" "Resistor_SMD:R_0402_1005Metric" (at 125.222 57.15 90)
+    (property "Footprint" "Library:R_0402_1005Metric" (at 125.222 57.15 90)
       (effects (font (size 1.27 1.27)) hide)
     )
@@
       (effects (font (size 1.27 1.27)) hide)
     )
-    (property "JLC" "0603" (at 127 57.15 0)
-      (effects (font (size 1.27 1.27)) hide)
-    )
-    (property "LCSC" "C22843" (at 127 57.15 0)
+    (property "JLC" "0402" (at 127 57.15 0)
+      (effects (font (size 1.27 1.27)) hide)
+    )
+    (property "LCSC" "C25867" (at 127 57.15 0)
       (effects (font (size 1.27 1.27)) hide)
     )
@@
       (effects (font (size 1.27 1.27)) (justify left))
     )
-    (property "Footprint" "Capacitor_SMD:C_0402_1005Metric" (at 127.9652 86.36 0)
+    (property "Footprint" "Library:C_0402_1005Metric" (at 127.9652 86.36 0)
       (effects (font (size 1.27 1.27)) hide)
     )
@@
       (effects (font (size 1.27 1.27)) (justify left))
     )
-    (property "Footprint" "Resistor_SMD:R_0402_1005Metric" (at 158.242 69.85 90)
+    (property "Footprint" "Library:R_0402_1005Metric" (at 158.242 69.85 90)
       (effects (font (size 1.27 1.27)) hide)
     )
@@
       (effects (font (size 1.27 1.27)) hide)
     )
-    (property "JLC" "0603" (at 160.02 69.85 0)
-      (effects (font (size 1.27 1.27)) hide)
-    )
-    (property "LCSC" "C22843" (at 160.02 69.85 0)
-      (effects (font (size 1.27 1.27)) hide)
-    )
+    (property "JLC" "0402" (at 160.02 69.85 0)
+      (effects (font (size 1.27 1.27)) hide)
+    )
+    (property "LCSC" "C25867" (at 160.02 69.85 0)
+      (effects (font (size 1.27 1.27)) hide)
+    )
