File: hardware/drake_10b/power_supply.kicad_sch (KiCad schematic)
At the start: 23 parts, among them J2 USB_C_Receptacle_USB2.0_16P, J3 Li-Ion, U2 XC6206P332MR-G, U3 TP4054

Commit message: revised production files
Parts:
- D16, D3: FT Rotation Offset (none) -> 180
- J2: FT Position Offset (none) -> 0,1.3335
- J3: FT Position Offset (none) -> 0.07,0.18; FT Rotation Offset (none) -> 180
- U3: FT Rotation Offset (none) -> 90; LCSC (none) -> C32574
Changed lines of the file:
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@@
+      (effects (font (size 1.27 1.27)) hide)
+    )
+    (property "FT Rotation Offset" "180" (at 139.7 147.32 0)
+      (effects (font (size 1.27 1.27)) hide)
+    )
+    (property "FT Position Offset" "0.07,0.18" (at 139.7 147.32 0)
       (effects (font (size 1.27 1.27)) hide)
     )
@@
       (effects (font (size 1.27 1.27)) hide)
     )
+    (property "FT Rotation Offset" "180" (at 124.46 72.39 90)
+      (effects (font (size 1.27 1.27)) hide)
+    )
     (pin "1")
     (pin "3")
@@
     )
     (property "LCSC" "C2931474" (at 96.52 50.8 0)
+      (effects (font (size 1.27 1.27)) hide)
+    )
+    (property "FT Position Offset" "0,1.3335" (at 96.52 50.8 0)
       (effects (font (size 1.27 1.27)) hide)
     )
@@
       (effects (font (size 1.27 1.27)) hide)
     )
+    (property "FT Rotation Offset" "180" (at 135.89 80.01 90)
+      (effects (font (size 1.27 1.27)) hide)
+    )
     (pin "1")
     (pin "3")
@@
       (effects (font (size 1.27 1.27)) hide)
     )
+    (property "LCSC" "C32574" (at 119.38 129.54 0)
+      (effects (font (size 1.27 1.27)) hide)
+    )
+    (property "FT Rotation Offset" "90" (at 119.38 129.54 0)
+      (effects (font (size 1.27 1.27)) hide)
+    )
