File: hardware/drake_10b/rear_light.kicad_sch (KiCad schematic)
At the start: 91 parts

Commit message: revised production files
Parts:
- JP1: LCSC C14033 -> C17168
Other:
- note added: "components on this sheet are only populated when using as light JP1 has to be populated, when using as 16 LED taillight"
Changed lines of the file:
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@@
     (stroke (width 0) (type default))
   )
+  (text "components on this sheet are only populated when using as light\n\nJP1 has to be populated, when using as 16 LED taillight"
+    (at 181.61 173.99 0)
+    (effects (font (size 1.27 1.27)) (justify left bottom))
+  )
   (hierarchical_label "START" (shape input) (at 36.83 71.12 180) (fields_autoplaced)
     (effects (font (size 1.27 1.27)) (justify right))
@@
       (effects (font (size 1.27 1.27)) hide)
     )
-    (property "LCSC" "C14033" (at 72.39 101.6 0)
+    (property "LCSC" "C17168" (at 72.39 101.6 0)
       (effects (font (size 1.27 1.27)) hide)
     )
